File: SignalForgeV4.kicad_sch (KiCad schematic)
At the start: 24 parts, among them J2 SPI_PINOUT, J3 I2C_PINOUT, J4 Conn_01x03_Socket, J5 BATTERY, J6 Micro_SD_Card_Det1, Q1 NPN, SW1 SW_SPDT, U1 ESP32-DEVKITC-32U, U2 USB_CHARGER_BOOST

Commit message: fix: update latest jlcpcb
Parts:
- added U3: DM-OLED096-636, DM-OLED096-636:MODULE_DM-OLED096-636, symbol DM-OLED096-636:DM-OLED096-636
- C_BTN1, D_BTN1, L_BTN1, R_BTN1, U_BTN1: footprint Button_Switch_SMD:SW_SPST_FSMSM -> Button_Switch_THT:SW_PUSH_1P1T_6x3.5mm_H5.0_APEM_MJTP1250
- D1: footprint (none) -> Connector_PinSocket_2.54mm:PinSocket_1x02_P2.54mm_Vertical
- J4: footprint (none) -> Connector_PinSocket_2.54mm:PinSocket_1x03_P2.54mm_Vertical
- J5: footprint (none) -> Connector_JST:JST_EH_S2B-EH_1x02_P2.50mm_Horizontal
- Q1: footprint (none) -> Package_TO_SOT_SMD:SOT-23_Handsoldering
- R1, R2: footprint (none) -> Resistor_SMD:R_0805_2012Metric_Pad1.20x1.40mm_HandSolder
- RN1: footprint Resistor_THT:R_Array_SIP5 -> Resistor_SMD:R_Array_Convex_4x0603
- RST_BTN1: footprint (none) -> Button_Switch_SMD:SW_SPST_FSMSM
Connections:
- net +3V3: now also J3.2 (Pin_2), U3.1 (GND); no longer J3.1 (Pin_1)
- net C_BTN: now also U1.8 (IO33); no longer U1.11 (IO27)
- net D_BTN: now also U1.11 (IO27); no longer U1.8 (IO33)
- net GND: now also J3.1 (Pin_1), U3.2 (VCC_IN); no longer J3.2 (Pin_2)
- net SCL: now also J3.4 (Pin_4), U3.3 (SCL); no longer J3.3 (Pin_3)
- net SDA: now also J3.3 (Pin_3), U3.4 (SDA); no longer J3.4 (Pin_4)
Other:
- note added: "**Note: VCC-GND Changed in Real Device"
